Commit message: lab 5

File: src/my_r2d2/urdf/r2d2.xacro (robot description, xacro)
@@ -219,9 +219,8 @@
       </geometry>
       <material name="black"/>
-      <origin xyz="0 0 0"/>
-    </visual>
-    <collision>
-      <geometry>
-        <cylinder radius="0.03" length="0.2"/>
+    </visual>
+    <collision>
+      <geometry>
+        <cylinder radius="0.03" length="0.1"/>
       </geometry>
     </collision>
@@ -233,3 +232,16 @@
      <origin rpy="0 1.57 0" xyz="0 0 0"/>
   </joint>
+ <link name="base_footprint">
+</link>
+<joint name="base_to_foot" type="fixed">
+    <parent link="base_footprint"/>
+    <child link="base_link"/>
+     <origin rpy="0 0 0" xyz="0 0 0.47"/>
+  </joint>
+ <link name="eye"></link>
+ <joint name="eye_to_lens" type="fixed">
+ <parent link="lens"/>
+ <child link="eye"/>
+ <origin rpy="0 0 -1.57" xyz="0 0 0"/>
+  </joint>
 </robot>
